File: EAGLEProjectFiles/DCDeluxe EAGLE/DCDeluxe.brd (EAGLE design)
At the start: 70 x 55 mm, 50 parts, among them IC1 STM32G431, IC2 LM386M-1, IC3 SRV05, IC4 7812T, IC5 78L33F

Commit message: TWEAKS:  Updated PCB layout
Parts:
- removed D3: 1N4004-M1, Duncs Diodes:SMA
- added B1: MB8S, rectifier:SOIC-4
- added TP13: TPTP20R, testpad:TP20R
- C16: value 47uF 50V -> 100uF 35V
- moved TP6 49.3 mm to (20.9, 2.86)
- moved TP9 38.4 mm to (51.6, 51.8)
- moved TP8 30.9 mm to (20.7, 52.0)
- moved TP3 14.3 mm to (28.2, 11.9)
- moved TP12 8.28 mm to (39.4, 22.9)
- moved TP10 6.36 mm to (26.7, 22.9)
- moved TP11 6.36 mm to (32.7, 22.9)
- moved TP5 6.19 mm to (15.9, 2.78)
- moved TP7 5.08 mm to (25.8, 51.9)
- moved VIN 1.19 mm to (18.4, 7.72)
- moved R1 0.96 mm to (62.2, 30.2)
- moved TP2 0.87 mm to (23.1, 11.9)
- moved C13 0.68 mm to (56.4, 2.28)
- moved C2 0.62 mm to (61.8, 39.7)
- moved TP4 0.43 mm to (53.1, 7.14)
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Connections:
- removed net N$14: C16.+, D3.K, IC4.1
- removed net VIN: D3.A, TP5.TP, VIN.2
- new net VIN+: B1.+, C16.+, IC4.1
- new net VIN1: B1.~1, TP5.TP, VIN.1
- new net VIN2: B1.~2, TP6.TP, VIN.2
- net GND: now also B1.-; no longer VIN.1
- net NRST: now also TP12.TP; no longer TP11.TP
- net SPK+: now also TP9.TP; no longer TP8.TP
- net SWCLK: now also TP11.TP; no longer TP10.TP
- net SWDIO: now also TP10.TP; no longer TP9.TP
- net TRIG1: now also TP7.TP; no longer TP6.TP
- net TRIG2: now also TP8.TP; no longer TP7.TP
- net VDDA: now also TP13.TP; no longer TP12.TP
Routing:
- net N$14: track 25.9 -> 0.00 mm, vias 1 -> 0
- net VIN+: track 0.00 -> 24.4 mm, vias 0 -> 1
- net VIN1: track 0.00 -> 15.0 mm
- net VIN2: track 0.00 -> 13.5 mm
- net VIN: track 10.3 -> 0.00 mm
- net +12V: track 53.0 -> 48.2 mm, vias 1 -> 2
- net GND: track 75.3 -> 71.4 mm
- net SPK+: track 20.1 -> 18.5 mm
- net N$2: track 11.1 -> 10.5 mm
- net VDD: track 48.2 -> 47.7 mm
- net N$4: track 26.0 -> 25.5 mm
