File: EAGLEProjectFiles/DCDeluxe EAGLE/DCDeluxe.sch (EAGLE design)
At the start: 50 parts, among them IC1 STM32G431, IC2 LM386M-1, IC3 SRV05, IC4 7812T, IC5 78L33F

Commit message: TWEAKS:  Updated PCB layout
Parts:
- removed D3: 1N4004-M1, Duncs Diodes:1N4004-M1
- added B1: MB8S, rectifier:MB8S
- added TP13: TPTP20R, testpad:TPTP20R
- C16: value 47uF 50V -> 100uF 35V
Connections:
- removed net N$14: C16.+, D3.K, IC4.VI
- removed net VIN: D3.A, TP5.TP, VIN-2.KL
- new net VIN+: B1.+, C16.+, IC4.VI
- new net VIN1: B1.AC1, TP5.TP, VIN-1.KL
- new net VIN2: B1.AC2, TP6.TP, VIN-2.KL
- net GND: now also B1.-; no longer VIN-1.KL
- net NRST: now also TP12.TP; no longer TP11.TP
- net SPK+: now also TP9.TP; no longer TP8.TP
- net SWCLK: now also TP11.TP; no longer TP10.TP
- net SWDIO: now also TP10.TP; no longer TP9.TP
- net TRIG1: now also TP7.TP; no longer TP6.TP
- net TRIG2: now also TP8.TP; no longer TP7.TP
- net VDDA: now also TP13.TP; no longer TP12.TP
Other:
- note added: "Choose either R4+R11 or R1"
- moved on the sheet: C4, R1, VIN-1, VIN-2
